File: board/board.kicad_pcb (KiCad board)
At the start: 2 copper layers, 21 x 13 mm, 1 part

Commit message: initial design
Parts:
- removed LOGO1: Logo_Open_Hardware_Small, Symbol:OSHW-Symbol_6.7x6mm_SilkScreen
- added C1: 12pF, Capacitor_SMD:C_0402_1005Metric, F.Cu at (151.6, 100.9)
- added C2: 12pF, Capacitor_SMD:C_0402_1005Metric, F.Cu at (154.1, 100.9)
- added C3: 100nF, Capacitor_SMD:C_0402_1005Metric, F.Cu at (146.0, 98.3)
- added C4: 1uF, Capacitor_SMD:C_0402_1005Metric, F.Cu at (147.0, 98.4)
- added J1: 001_I2C, on_edge:on_edge_2x05_device, F.Cu at (140.0, 96.5)
- added J2: 001_I2C, on_edge:on_edge_2x05_host, F.Cu at (161.0, 96.5)
- added U1: PCF8563T, Package_SO:SOIC-8_3.9x4.9mm_P1.27mm, F.Cu at (149.1, 94.6)
- added Y1: 32.768kHz, Crystal:Crystal_SMD_3215-2Pin_3.2x1.5mm, F.Cu at (152.8, 98.6)
Routing:
- net GND: track 0.00 -> 32.9 mm
- net /rtc/~{INT}: track 0.00 -> 26.7 mm, vias 0 -> 2
- net /rtc/SCL: track 0.00 -> 22.3 mm, vias 0 -> 2
- net /rtc/VDD: track 0.00 -> 19.8 mm, vias 0 -> 1
- net /rtc/SDA: track 0.00 -> 19.4 mm, vias 0 -> 2
- net Net-(J1-N/C): track 0.00 -> 17.2 mm, vias 0 -> 2
- net Net-(J1-5V): track 0.00 -> 17.2 mm
- net Net-(J1-status): track 0.00 -> 16.6 mm
- net Net-(J1-CS/EN): track 0.00 -> 16.2 mm
- net Net-(J1-~{RESET}): track 0.00 -> 16.1 mm
- net Net-(U1-OSCO): track 0.00 -> 6.38 mm
- net Net-(U1-OSCI): track 0.00 -> 3.89 mm
Other:
- outline, holes or cut-outs redrawn
- board text added: "osf.001"
- board text added: "osf.b158.v1.0"
