File: board/board.kicad_sch (KiCad schematic)
At the start: 1 part

Commit message: initial design
Parts:
- added J1: 001_I2C, on_edge:on_edge_2x05_device, symbol put_on_edge:001_I2C
- added J2: 001_I2C, on_edge:on_edge_2x05_host, symbol put_on_edge:001_I2C
Connections:
- net GND: now also J1.1 (GND), J2.1 (GND)
- new net: J1.10 (5V), J2.10 (5V)
- new net: J1.3 (N/C), J2.3 (N/C)
- new net: J1.6 (CS/EN), J2.6 (CS/EN)
- new net: J1.7 (status), J2.7 (status)
- new net: J1.8 (~{RESET}), J2.8 (~{RESET})
- new net rtc/SCL: J1.4 (SCL), J2.4 (SCL)
- new net rtc/SDA: J1.2 (SDA), J2.2 (SDA)
- new net rtc/VDD: J1.9 (3.3V), J2.9 (3.3V)
- new net rtc/~{INT}: J1.5 (INT), J2.5 (INT)
- no-connect marks 0 -> 1
Other:
- removed sheet implementation
- added sheet rtc (rtc.kicad_sch)
- note removed: "Input connectors go here"
- note removed: "Output connectors go here"
